File: hardware/circle-main/legacy/02_power.sch (KiCad schematic (older format))
At the start: 23 parts, among them J2 LIPO_1S_NTC, Q1 SD_RAIL_SWITCH, Q2 PPG_LED_RAIL_SWITCH, Q3 HAPTIC_RAIL_SWITCH, Q4 ISOLATION_RAIL_SWITCH, Q5 EXPANSION_RAIL_SWITCH, U2 BQ24074, U3 TPS63070, U4 TPS3700, U5 TPS3700

Commit message: Make every CIRCLE review claim reproducible
Validate and export the architecture-level schematics with KiCad 10.0.5, add zero-violation ERC gates, engineering documentation, and one-command evidence hashing.

Constraint: KiCad CLI does not import legacy .sch into native .kicad_sch

Rejected: Hand-written native S-expressions | would create unvalidated CAD

Confidence: medium

Scope-risk: broad

Reversibility: clean

Directive: Treat NET annotations as architecture interfaces, not fabrication-ready connectivity

Tested: py -3.11 tools/verify_release.py; 30 tests; KiCad 10.0.5 ERC/BOM/PDF/SVG/netlist exports

Not-tested: Native conversion, PCB layout, footprints, powered electrodes, human connection, EMC, or regulatory compliance
Other:
- note added: "NET:BATTERY_VALID"
- note added: "NET:SAFETY_POWER_GOOD"
- note added: "NET:SW_EXPANSION"
- note added: "NET:SW_HAPTIC"
- note added: "NET:SW_ISOLATION"
- note added: "NET:SW_PPG_LED"
- note added: "NET:SW_SD"
- note added: "NET:USB_PRESENT"
- note added: "NET:VBAT"
- note added: "NET:VBUS_5V"
Changed lines of the file:
@@
 Sheet 1 1
 Title "Battery, charging, and partitioned rails"
+Date "2026-08-14"
+Rev "A"
+Comp "Vers3Dynamics"
 Comment1 "ENGINEERING REVIEW ONLY - NOT FOR HUMAN CONNECTION"
+Comment2 "Generated artifact - edit manifest/generator"
+Comment3 ""
+Comment4 ""
 $EndDescr
 $Comp
@@
 F 0 "U2" H 1400 1300 50  0000 C CNN
 F 1 "BQ24074" H 1400 1100 50  0000 C CNN
+F 2 "" H 1300 1200 50  0001 C CNN
+F 3 "" H 1300 1200 50  0001 C CNN
+	1    1300 1200
 	1    0    0    -1
 $EndComp
@@
 F 0 "U3" H 3500 1300 50  0000 C CNN
 F 1 "TPS63070" H 3500 1100 50  0000 C CNN
+F 2 "" H 3400 1200 50  0001 C CNN
+F 3 "" H 3400 1200 50  0001 C CNN
+	1    3400 1200
 	1    0    0    -1
 $EndComp
@@
 F 0 "U4" H 5600 1300 50  0000 C CNN
 F 1 "TPS3700" H 5600 1100 50  0000 C CNN
+F 2 "" H 5500 1200 50  0001 C CNN
+F 3 "" H 5500 1200 50  0001 C CNN
+	1    5500 1200
 	1    0    0    -1
 $EndComp
@@
 F 0 "U5" H 7700 1300 50  0000 C CNN
 F 1 "TPS3700" H 7700 1100 50  0000 C CNN
+F 2 "" H 7600 1200 50  0001 C CNN
+F 3 "" H 7600 1200 50  0001 C CNN
+	1    7600 1200
 	1    0    0    -1
 $EndComp
@@
 F 0 "J2" H 1400 2100 50  0000 C CNN
 F 1 "LIPO_1S_NTC" H 1400 1900 50  0000 C CNN
+F 2 "" H 1300 2000 50  0001 C CNN
+F 3 "" H 1300 2000 50  0001 C CNN
+	1    1300 2000
 	1    0    0    -1
 $EndComp
@@
 F 0 "F1" H 3500 2100 50  0000 C CNN
 F 1 "USB_INPUT_FUSE" H 3500 1900 50  0000 C CNN
+F 2 "" H 3400 2000 50  0001 C CNN
+F 3 "" H 3400 2000 50  0001 C CNN
+	1    3400 2000
 	1    0    0    -1
 $EndComp
@@
 F 0 "Q1" H 5600 2100 50  0000 C CNN
 F 1 "SD_RAIL_SWITCH" H 5600 1900 50  0000 C CNN
+F 2 "" H 5500 2000 50  0001 C CNN
+F 3 "" H 5500 2000 50  0001 C CNN
+	1    5500 2000
 	1    0    0    -1
 $EndComp
@@
 F 0 "Q2" H 7700 2100 50  0000 C CNN
 F 1 "PPG_LED_RAIL_SWITCH" H 7700 1900 50  0000 C CNN
+F 2 "" H 7600 2000 50  0001 C CNN
+F 3 "" H 7600 2000 50  0001 C CNN
+	1    7600 2000
 	1    0    0    -1
 $EndComp
@@
 F 0 "Q3" H 1400 2900 50  0000 C CNN
 F 1 "HAPTIC_RAIL_SWITCH" H 1400 2700 50  0000 C CNN
+F 2 "" H 1300 2800 50  0001 C CNN
+F 3 "" H 1300 2800 50  0001 C CNN
+	1    1300 2800
 	1    0    0    -1
 $EndComp
@@
 F 0 "Q4" H 3500 2900 50  0000 C CNN
 F 1 "ISOLATION_RAIL_SWITCH" H 3500 2700 50  0000 C CNN
+F 2 "" H 3400 2800 50  0001 C CNN
+F 3 "" H 3400 2800 50  0001 C CNN
+	1    3400 2800
 	1    0    0    -1
 $EndComp
@@
 F 0 "Q5" H 5600 2900 50  0000 C CNN
 F 1 "EXPANSION_RAIL_SWITCH" H 5600 2700 50  0000 C CNN
+F 2 "" H 5500 2800 50  0001 C CNN
+F 3 "" H 5500 2800 50  0001 C CNN
+	1    5500 2800
 	1    0    0    -1
 $EndComp
@@
 F 0 "RSH1" H 7700 2900 50  0000 C CNN
 F 1 "CURRENT_SHUNT" H 7700 2700 50  0000 C CNN
+F 2 "" H 7600 2800 50  0001 C CNN
+F 3 "" H 7600 2800 50  0001 C CNN
+	1    7600 2800
 	1    0    0    -1
 $EndComp
@@
 F 0 "RSH2" H 1400 3700 50  0000 C CNN
 F 1 "CURRENT_SHUNT" H 1400 3500 50  0000 C CNN
+F 2 "" H 1300 3600 50  0001 C CNN
+F 3 "" H 1300 3600 50  0001 C CNN
+	1    1300 3600
 	1    0    0    -1
 $EndComp
@@
 F 0 "RSH3" H 3500 3700 50  0000 C CNN
 F 1 "CURRENT_SHUNT" H 3500 3500 50  0000 C CNN
+F 2 "" H 3400 3600 50  0001 C CNN
+F 3 "" H 3400 3600 50  0001 C CNN
+	1    3400 3600
 	1    0    0    -1
 $EndComp
@@
 F 0 "RSH4" H 5600 3700 50  0000 C CNN
 F 1 "CURRENT_SHUNT" H 5600 3500 50  0000 C CNN
+F 2 "" H 5500 3600 50  0001 C CNN
+F 3 "" H 5500 3600 50  0001 C CNN
+	1    5500 3600
 	1    0    0    -1
 $EndComp
@@
 F 0 "RSH5" H 7700 3700 50  0000 C CNN
 F 1 "CURRENT_SHUNT" H 7700 3500 50  0000 C CNN
+F 2 "" H 7600 3600 50  0001 C CNN
+F 3 "" H 7600 3600 50  0001 C CNN
+	1    7600 3600
 	1    0    0    -1
 $EndComp
@@
 F 0 "RSH6" H 1400 4500 50  0000 C CNN
 F 1 "CURRENT_SHUNT" H 1400 4300 50  0000 C CNN
+F 2 "" H 1300 4400 50  0001 C CNN
+F 3 "" H 1300 4400 50  0001 C CNN
+	1    1300 4400
 	1    0    0    -1
 $EndComp
@@
 F 0 "JP1" H 3500 4500 50  0000 C CNN
 F 1 "KELVIN_MEASURE_JUMPER" H 3500 4300 50  0000 C CNN
+F 2 "" H 3400 4400 50  0001 C CNN
+F 3 "" H 3400 4400 50  0001 C CNN
+	1    3400 4400
 	1    0    0    -1
 $EndComp
@@
 F 0 "JP2" H 5600 4500 50  0000 C CNN
 F 1 "KELVIN_MEASURE_JUMPER" H 5600 4300 50  0000 C CNN
+F 2 "" H 5500 4400 50  0001 C CNN
+F 3 "" H 5500 4400 50  0001 C CNN
+	1    5500 4400
 	1    0    0    -1
 $EndComp
@@
 F 0 "JP3" H 7700 4500 50  0000 C CNN
 F 1 "KELVIN_MEASURE_JUMPER" H 7700 4300 50  0000 C CNN
+F 2 "" H 7600 4400 50  0001 C CNN
+F 3 "" H 7600 4400 50  0001 C CNN
+	1    7600 4400
 	1    0    0    -1
 $EndComp
@@
 F 0 "JP4" H 1400 5300 50  0000 C CNN
 F 1 "KELVIN_MEASURE_JUMPER" H 1400 5100 50  0000 C CNN
+F 2 "" H 1300 5200 50  0001 C CNN
+F 3 "" H 1300 5200 50  0001 C CNN
+	1    1300 5200
 	1    0    0    -1
 $EndComp
@@
 F 0 "JP5" H 3500 5300 50  0000 C CNN
 F 1 "KELVIN_MEASURE_JUMPER" H 3500 5100 50  0000 C CNN
+F 2 "" H 3400 5200 50  0001 C CNN
+F 3 "" H 3400 5200 50  0001 C CNN
+	1    3400 5200
 	1    0    0    -1
 $EndComp
@@
 F 0 "JP6" H 5600 5300 50  0000 C CNN
 F 1 "KELVIN_MEASURE_JUMPER" H 5600 5100 50  0000 C CNN
-	1    0    0    -1
-$EndComp
-Text Label 700 5600 0    50   ~ 0
-VBUS_5V
-Text Label 700 5840 0    50   ~ 0
-USB_PRESENT
-Text Label 700 6080 0    50   ~ 0
-VBAT
-Text Label 700 6320 0    50   ~ 0
-BATTERY_VALID
-Text Label 700 6560 0    50   ~ 0
-SAFETY_POWER_GOOD
-Text Label 700 6800 0    50   ~ 0
-SW_SD
-Text Label 700 7040 0    50   ~ 0
-SW_PPG_LED
-Text Label 700 7280 0    50   ~ 0
-SW_HAPTIC
-Text Label 6000 5600 0    50   ~ 0
-SW_ISOLATION
-Text Label 6000 5840 0    50   ~ 0
-SW_EXPANSION
+F 2 "" H 5500 5200 50  0001 C CNN
+F 3 "" H 5500 5200 50  0001 C CNN
+	1    5500 5200
+	1    0    0    -1
+$EndComp
 Text Notes 600 400 0    50   ~ 0
 ENGINEERING REVIEW ONLY - NOT FOR HUMAN CONNECTION
+Text Notes 700 5600 0    50   ~ 0
+NET:VBUS_5V
+Text Notes 700 5850 0    50   ~ 0
+NET:USB_PRESENT
+Text Notes 700 6100 0    50   ~ 0
+NET:VBAT
+Text Notes 700 6350 0    50   ~ 0
+NET:BATTERY_VALID
+Text Notes 700 6600 0    50   ~ 0
+NET:SAFETY_POWER_GOOD
+Text Notes 700 6850 0    50   ~ 0
+NET:SW_SD
+Text Notes 700 7100 0    50   ~ 0
+NET:SW_PPG_LED
+Text Notes 700 7350 0    50   ~ 0
+NET:SW_HAPTIC
+Text Notes 6000 5600 0    50   ~ 0
+NET:SW_ISOLATION
+Text Notes 6000 5850 0    50   ~ 0
+NET:SW_EXPANSION
 $EndSCHEMATC
