File: hardware/circle-main/legacy/03_eda_safety.sch (KiCad schematic (older format))
At the start: 14 parts, among them J10 EDA_ELECTRODES, J11 CAL_INJECTION_BEHIND_LIMITS, K1 REVIEW_GATE:EDA_SWITCH_SELECT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, K2 REVIEW_GATE:EDA_SWITCH_SELECT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, U10 ADS1220, U11 OPA2192, U12 REF5020, U13 TPS3700, U14 TPS3700, U15 TPS3700

Commit message: Make every CIRCLE review claim reproducible
Validate and export the architecture-level schematics with KiCad 10.0.5, add zero-violation ERC gates, engineering documentation, and one-command evidence hashing.

Constraint: KiCad CLI does not import legacy .sch into native .kicad_sch

Rejected: Hand-written native S-expressions | would create unvalidated CAD

Confidence: medium

Scope-risk: broad

Reversibility: clean

Directive: Treat NET annotations as architecture interfaces, not fabrication-ready connectivity

Tested: py -3.11 tools/verify_release.py; 30 tests; KiCad 10.0.5 ERC/BOM/PDF/SVG/netlist exports

Not-tested: Native conversion, PCB layout, footprints, powered electrodes, human connection, EMC, or regulatory compliance
Other:
- note added: "NET:DEBUG_ATTACHED"
- note added: "NET:EDA_ACTIVE"
- note added: "NET:EDA_ANALOG_GOOD"
- note added: "NET:EDA_FW_REQUEST"
- note added: "NET:EDA_PREPARE"
- note added: "NET:EXTERNAL_EXPANSION_ATTACHED"
- note added: "NET:USB_PRESENT"
Changed lines of the file:
@@
 Sheet 1 1
 Title "EDA acquisition and fail-off interlocks"
+Date "2026-08-14"
+Rev "A"
+Comp "Vers3Dynamics"
 Comment1 "ENGINEERING REVIEW ONLY - NOT FOR HUMAN CONNECTION"
+Comment2 "Generated artifact - edit manifest/generator"
+Comment3 ""
+Comment4 ""
 $EndDescr
 $Comp
@@
 F 0 "U10" H 1400 1300 50  0000 C CNN
 F 1 "ADS1220" H 1400 1100 50  0000 C CNN
+F 2 "" H 1300 1200 50  0001 C CNN
+F 3 "" H 1300 1200 50  0001 C CNN
+	1    1300 1200
 	1    0    0    -1
 $EndComp
@@
 F 0 "U11" H 3500 1300 50  0000 C CNN
 F 1 "OPA2192" H 3500 1100 50  0000 C CNN
+F 2 "" H 3400 1200 50  0001 C CNN
+F 3 "" H 3400 1200 50  0001 C CNN
+	1    3400 1200
 	1    0    0    -1
 $EndComp
@@
 F 0 "U12" H 5600 1300 50  0000 C CNN
 F 1 "REF5020" H 5600 1100 50  0000 C CNN
+F 2 "" H 5500 1200 50  0001 C CNN
+F 3 "" H 5500 1200 50  0001 C CNN
+	1    5500 1200
 	1    0    0    -1
 $EndComp
@@
 F 0 "U13" H 7700 1300 50  0000 C CNN
 F 1 "TPS3700" H 7700 1100 50  0000 C CNN
+F 2 "" H 7600 1200 50  0001 C CNN
+F 3 "" H 7600 1200 50  0001 C CNN
+	1    7600 1200
 	1    0    0    -1
 $EndComp
@@
 F 0 "U14" H 1400 2100 50  0000 C CNN
 F 1 "TPS3700" H 1400 1900 50  0000 C CNN
+F 2 "" H 1300 2000 50  0001 C CNN
+F 3 "" H 1300 2000 50  0001 C CNN
+	1    1300 2000
 	1    0    0    -1
 $EndComp
@@
 F 0 "U15" H 3500 2100 50  0000 C CNN
 F 1 "TPS3700" H 3500 1900 50  0000 C CNN
+F 2 "" H 3400 2000 50  0001 C CNN
+F 3 "" H 3400 2000 50  0001 C CNN
+	1    3400 2000
 	1    0    0    -1
 $EndComp
@@
 F 0 "K1" H 5600 2100 50  0000 C CNN
 F 1 "REVIEW_GATE:EDA_SWITCH_SELECTION" H 5600 1900 50  0000 C CNN
+F 2 "" H 5500 2000 50  0001 C CNN
+F 3 "" H 5500 2000 50  0001 C CNN
+	1    5500 2000
 	1    0    0    -1
 $EndComp
@@
 F 0 "K2" H 7700 2100 50  0000 C CNN
 F 1 "REVIEW_GATE:EDA_SWITCH_SELECTION" H 7700 1900 50  0000 C CNN
+F 2 "" H 7600 2000 50  0001 C CNN
+F 3 "" H 7600 2000 50  0001 C CNN
+	1    7600 2000
 	1    0    0    -1
 $EndComp
@@
 F 0 "R_EDA_A1" H 1400 2900 50  0000 C CNN
 F 1 "REVIEW_GATE:EDA_LIMIT_NETWORK" H 1400 2700 50  0000 C CNN
+F 2 "" H 1300 2800 50  0001 C CNN
+F 3 "" H 1300 2800 50  0001 C CNN
+	1    1300 2800
 	1    0    0    -1
 $EndComp
@@
 F 0 "R_EDA_A2" H 3500 2900 50  0000 C CNN
 F 1 "REVIEW_GATE:EDA_LIMIT_NETWORK" H 3500 2700 50  0000 C CNN
+F 2 "" H 3400 2800 50  0001 C CNN
+F 3 "" H 3400 2800 50  0001 C CNN
+	1    3400 2800
 	1    0    0    -1
 $EndComp
@@
 F 0 "R_EDA_B1" H 5600 2900 50  0000 C CNN
 F 1 "REVIEW_GATE:EDA_LIMIT_NETWORK" H 5600 2700 50  0000 C CNN
+F 2 "" H 5500 2800 50  0001 C CNN
+F 3 "" H 5500 2800 50  0001 C CNN
+	1    5500 2800
 	1    0    0    -1
 $EndComp
@@
 F 0 "R_EDA_B2" H 7700 2900 50  0000 C CNN
 F 1 "REVIEW_GATE:EDA_LIMIT_NETWORK" H 7700 2700 50  0000 C CNN
+F 2 "" H 7600 2800 50  0001 C CNN
+F 3 "" H 7600 2800 50  0001 C CNN
+	1    7600 2800
 	1    0    0    -1
 $EndComp
@@
 F 0 "J10" H 1400 3700 50  0000 C CNN
 F 1 "EDA_ELECTRODES" H 1400 3500 50  0000 C CNN
+F 2 "" H 1300 3600 50  0001 C CNN
+F 3 "" H 1300 3600 50  0001 C CNN
+	1    1300 3600
 	1    0    0    -1
 $EndComp
@@
 F 0 "J11" H 3500 3700 50  0000 C CNN
 F 1 "CAL_INJECTION_BEHIND_LIMITS" H 3500 3500 50  0000 C CNN
+F 2 "" H 3400 3600 50  0001 C CNN
+F 3 "" H 3400 3600 50  0001 C CNN
+	1    3400 3600
 	1    0    0    -1
 $EndComp
-Text Label 700 5600 0    50   ~ 0
-EDA_PREPARE
-Text Label 700 5840 0    50   ~ 0
-EDA_ACTIVE
-Text Label 700 6080 0    50   ~ 0
-EDA_ANALOG_GOOD
-Text Label 700 6320 0    50   ~ 0
-USB_PRESENT
-Text Label 700 6560 0    50   ~ 0
-DEBUG_ATTACHED
-Text Label 700 6800 0    50   ~ 0
-EXTERNAL_EXPANSION_ATTACHED
-Text Label 700 7040 0    50   ~ 0
-EDA_FW_REQUEST
 Text Notes 600 400 0    50   ~ 0
 ENGINEERING REVIEW ONLY - NOT FOR HUMAN CONNECTION
-Text Notes 700 7280 0    50   ~ 0
+Text Notes 700 5600 0    50   ~ 0
+NET:EDA_PREPARE
+Text Notes 700 5850 0    50   ~ 0
+NET:EDA_ACTIVE
+Text Notes 700 6100 0    50   ~ 0
+NET:EDA_ANALOG_GOOD
+Text Notes 700 6350 0    50   ~ 0
+NET:USB_PRESENT
+Text Notes 700 6600 0    50   ~ 0
+NET:DEBUG_ATTACHED
+Text Notes 700 6850 0    50   ~ 0
+NET:EXTERNAL_EXPANSION_ATTACHED
+Text Notes 700 7100 0    50   ~ 0
+NET:EDA_FW_REQUEST
+Text Notes 700 7350 0    50   ~ 0
 REVIEW_GATE:EDA_LIMIT_NETWORK
 Text Notes 6000 5600 0    50   ~ 0
 REVIEW_GATE:EDA_SWITCH_SELECTION
-Text Notes 6000 5840 0    50   ~ 0
+Text Notes 6000 5850 0    50   ~ 0
 PASSIVE LIMITS REMAIN SERIES UNDER ONE WELDED SWITCH
 $EndSCHEMATC
