File: hardware/circle-main/legacy/05_storage.sch (KiCad schematic (older format))
At the start: 9 parts, among them J21 MICROSD_4BIT_CARD_DETECT

Commit message: Make every CIRCLE review claim reproducible
Validate and export the architecture-level schematics with KiCad 10.0.5, add zero-violation ERC gates, engineering documentation, and one-command evidence hashing.

Constraint: KiCad CLI does not import legacy .sch into native .kicad_sch

Rejected: Hand-written native S-expressions | would create unvalidated CAD

Confidence: medium

Scope-risk: broad

Reversibility: clean

Directive: Treat NET annotations as architecture interfaces, not fabrication-ready connectivity

Tested: py -3.11 tools/verify_release.py; 30 tests; KiCad 10.0.5 ERC/BOM/PDF/SVG/netlist exports

Not-tested: Native conversion, PCB layout, footprints, powered electrodes, human connection, EMC, or regulatory compliance
Other:
- note added: "NET:SAFE_EJECT"
- note added: "NET:SD_CARD_DETECT"
- note added: "NET:SD_CLK"
- note added: "NET:SD_CMD"
- note added: "NET:SD_D0"
- note added: "NET:SD_D1"
- note added: "NET:SD_D2"
- note added: "NET:SD_D3"
Changed lines of the file:
@@
 Sheet 1 1
 Title "4-bit SDMMC recorder"
+Date "2026-08-14"
+Rev "A"
+Comp "Vers3Dynamics"
 Comment1 "ENGINEERING REVIEW ONLY - NOT FOR HUMAN CONNECTION"
+Comment2 "Generated artifact - edit manifest/generator"
+Comment3 ""
+Comment4 ""
 $EndDescr
 $Comp
@@
 F 0 "J21" H 1400 1300 50  0000 C CNN
 F 1 "MICROSD_4BIT_CARD_DETECT" H 1400 1100 50  0000 C CNN
+F 2 "" H 1300 1200 50  0001 C CNN
+F 3 "" H 1300 1200 50  0001 C CNN
+	1    1300 1200
 	1    0    0    -1
 $EndComp
@@
 F 0 "D21" H 3500 1300 50  0000 C CNN
 F 1 "SD_ESD_BAT_DOMAIN" H 3500 1100 50  0000 C CNN
+F 2 "" H 3400 1200 50  0001 C CNN
+F 3 "" H 3400 1200 50  0001 C CNN
+	1    3400 1200
 	1    0    0    -1
 $EndComp
@@
 F 0 "S20" H 5600 1300 50  0000 C CNN
 F 1 "SAFE_EJECT" H 5600 1100 50  0000 C CNN
+F 2 "" H 5500 1200 50  0001 C CNN
+F 3 "" H 5500 1200 50  0001 C CNN
+	1    5500 1200
 	1    0    0    -1
 $EndComp
@@
 F 0 "RSD1" H 7700 1300 50  0000 C CNN
 F 1 "SDMMC_SERIES_DAMPING" H 7700 1100 50  0000 C CNN
+F 2 "" H 7600 1200 50  0001 C CNN
+F 3 "" H 7600 1200 50  0001 C CNN
+	1    7600 1200
 	1    0    0    -1
 $EndComp
@@
 F 0 "RSD2" H 1400 2100 50  0000 C CNN
 F 1 "SDMMC_SERIES_DAMPING" H 1400 1900 50  0000 C CNN
+F 2 "" H 1300 2000 50  0001 C CNN
+F 3 "" H 1300 2000 50  0001 C CNN
+	1    1300 2000
 	1    0    0    -1
 $EndComp
@@
 F 0 "RSD3" H 3500 2100 50  0000 C CNN
 F 1 "SDMMC_SERIES_DAMPING" H 3500 1900 50  0000 C CNN
+F 2 "" H 3400 2000 50  0001 C CNN
+F 3 "" H 3400 2000 50  0001 C CNN
+	1    3400 2000
 	1    0    0    -1
 $EndComp
@@
 F 0 "RSD4" H 5600 2100 50  0000 C CNN
 F 1 "SDMMC_SERIES_DAMPING" H 5600 1900 50  0000 C CNN
+F 2 "" H 5500 2000 50  0001 C CNN
+F 3 "" H 5500 2000 50  0001 C CNN
+	1    5500 2000
 	1    0    0    -1
 $EndComp
@@
 F 0 "RSD5" H 7700 2100 50  0000 C CNN
 F 1 "SDMMC_SERIES_DAMPING" H 7700 1900 50  0000 C CNN
+F 2 "" H 7600 2000 50  0001 C CNN
+F 3 "" H 7600 2000 50  0001 C CNN
+	1    7600 2000
 	1    0    0    -1
 $EndComp
@@
 F 0 "RSD6" H 1400 2900 50  0000 C CNN
 F 1 "SDMMC_SERIES_DAMPING" H 1400 2700 50  0000 C CNN
+F 2 "" H 1300 2800 50  0001 C CNN
+F 3 "" H 1300 2800 50  0001 C CNN
+	1    1300 2800
 	1    0    0    -1
 $EndComp
-Text Label 700 5600 0    50   ~ 0
-SD_D0
-Text Label 700 5840 0    50   ~ 0
-SD_D1
-Text Label 700 6080 0    50   ~ 0
-SD_D2
-Text Label 700 6320 0    50   ~ 0
-SD_D3
-Text Label 700 6560 0    50   ~ 0
-SD_CLK
-Text Label 700 6800 0    50   ~ 0
-SD_CMD
-Text Label 700 7040 0    50   ~ 0
-SD_CARD_DETECT
-Text Label 700 7280 0    50   ~ 0
-SAFE_EJECT
 Text Notes 600 400 0    50   ~ 0
 ENGINEERING REVIEW ONLY - NOT FOR HUMAN CONNECTION
+Text Notes 700 5600 0    50   ~ 0
+NET:SD_D0
+Text Notes 700 5850 0    50   ~ 0
+NET:SD_D1
+Text Notes 700 6100 0    50   ~ 0
+NET:SD_D2
+Text Notes 700 6350 0    50   ~ 0
+NET:SD_D3
+Text Notes 700 6600 0    50   ~ 0
+NET:SD_CLK
+Text Notes 700 6850 0    50   ~ 0
+NET:SD_CMD
+Text Notes 700 7100 0    50   ~ 0
+NET:SD_CARD_DETECT
+Text Notes 700 7350 0    50   ~ 0
+NET:SAFE_EJECT
 Text Notes 6000 5600 0    50   ~ 0
 ASYNCHRONOUS STORAGE NEVER BLOCKS CAPTURE
