File: hardware/circle-main/legacy/08_observability.sch (KiCad schematic (older format))
At the start: 16 parts

Commit message: Make every CIRCLE review claim reproducible
Validate and export the architecture-level schematics with KiCad 10.0.5, add zero-violation ERC gates, engineering documentation, and one-command evidence hashing.

Constraint: KiCad CLI does not import legacy .sch into native .kicad_sch

Rejected: Hand-written native S-expressions | would create unvalidated CAD

Confidence: medium

Scope-risk: broad

Reversibility: clean

Directive: Treat NET annotations as architecture interfaces, not fabrication-ready connectivity

Tested: py -3.11 tools/verify_release.py; 30 tests; KiCad 10.0.5 ERC/BOM/PDF/SVG/netlist exports

Not-tested: Native conversion, PCB layout, footprints, powered electrodes, human connection, EMC, or regulatory compliance
Other:
- note added: "NET:FAULT_INJECTION"
- note added: "NET:TP_ALL_RAILS"
- note added: "NET:TP_BATTERY_VALID"
- note added: "NET:TP_EDA_ANALOG_GOOD"
- note added: "NET:TP_SAFETY_POWER_GOOD"
- note added: "NET:TP_SD_ACTIVITY"
- note added: "NET:TP_SYNC_BOTH_SIDES"
- note added: "NET:TP_USB_PRESENT"
Changed lines of the file:
@@
 Sheet 1 1
 Title "Test points and fault injection"
+Date "2026-08-14"
+Rev "A"
+Comp "Vers3Dynamics"
 Comment1 "ENGINEERING REVIEW ONLY - NOT FOR HUMAN CONNECTION"
+Comment2 "Generated artifact - edit manifest/generator"
+Comment3 ""
+Comment4 ""
 $EndDescr
 $Comp
@@
 F 0 "TP1" H 1400 1300 50  0000 C CNN
 F 1 "RAIL_OR_SAFETY_TEST_POINT" H 1400 1100 50  0000 C CNN
+F 2 "" H 1300 1200 50  0001 C CNN
+F 3 "" H 1300 1200 50  0001 C CNN
+	1    1300 1200
 	1    0    0    -1
 $EndComp
@@
 F 0 "TP2" H 3500 1300 50  0000 C CNN
 F 1 "RAIL_OR_SAFETY_TEST_POINT" H 3500 1100 50  0000 C CNN
+F 2 "" H 3400 1200 50  0001 C CNN
+F 3 "" H 3400 1200 50  0001 C CNN
+	1    3400 1200
 	1    0    0    -1
 $EndComp
@@
 F 0 "TP3" H 5600 1300 50  0000 C CNN
 F 1 "RAIL_OR_SAFETY_TEST_POINT" H 5600 1100 50  0000 C CNN
+F 2 "" H 5500 1200 50  0001 C CNN
+F 3 "" H 5500 1200 50  0001 C CNN
+	1    5500 1200
 	1    0    0    -1
 $EndComp
@@
 F 0 "TP4" H 7700 1300 50  0000 C CNN
 F 1 "RAIL_OR_SAFETY_TEST_POINT" H 7700 1100 50  0000 C CNN
+F 2 "" H 7600 1200 50  0001 C CNN
+F 3 "" H 7600 1200 50  0001 C CNN
+	1    7600 1200
 	1    0    0    -1
 $EndComp
@@
 F 0 "TP5" H 1400 2100 50  0000 C CNN
 F 1 "RAIL_OR_SAFETY_TEST_POINT" H 1400 1900 50  0000 C CNN
+F 2 "" H 1300 2000 50  0001 C CNN
+F 3 "" H 1300 2000 50  0001 C CNN
+	1    1300 2000
 	1    0    0    -1
 $EndComp
@@
 F 0 "TP6" H 3500 2100 50  0000 C CNN
 F 1 "RAIL_OR_SAFETY_TEST_POINT" H 3500 1900 50  0000 C CNN
+F 2 "" H 3400 2000 50  0001 C CNN
+F 3 "" H 3400 2000 50  0001 C CNN
+	1    3400 2000
 	1    0    0    -1
 $EndComp
@@
 F 0 "TP7" H 5600 2100 50  0000 C CNN
 F 1 "RAIL_OR_SAFETY_TEST_POINT" H 5600 1900 50  0000 C CNN
+F 2 "" H 5500 2000 50  0001 C CNN
+F 3 "" H 5500 2000 50  0001 C CNN
+	1    5500 2000
 	1    0    0    -1
 $EndComp
@@
 F 0 "TP8" H 7700 2100 50  0000 C CNN
 F 1 "RAIL_OR_SAFETY_TEST_POINT" H 7700 1900 50  0000 C CNN
+F 2 "" H 7600 2000 50  0001 C CNN
+F 3 "" H 7600 2000 50  0001 C CNN
+	1    7600 2000
 	1    0    0    -1
 $EndComp
@@
 F 0 "TP9" H 1400 2900 50  0000 C CNN
 F 1 "RAIL_OR_SAFETY_TEST_POINT" H 1400 2700 50  0000 C CNN
+F 2 "" H 1300 2800 50  0001 C CNN
+F 3 "" H 1300 2800 50  0001 C CNN
+	1    1300 2800
 	1    0    0    -1
 $EndComp
@@
 F 0 "TP10" H 3500 2900 50  0000 C CNN
 F 1 "RAIL_OR_SAFETY_TEST_POINT" H 3500 2700 50  0000 C CNN
+F 2 "" H 3400 2800 50  0001 C CNN
+F 3 "" H 3400 2800 50  0001 C CNN
+	1    3400 2800
 	1    0    0    -1
 $EndComp
@@
 F 0 "TP11" H 5600 2900 50  0000 C CNN
 F 1 "RAIL_OR_SAFETY_TEST_POINT" H 5600 2700 50  0000 C CNN
+F 2 "" H 5500 2800 50  0001 C CNN
+F 3 "" H 5500 2800 50  0001 C CNN
+	1    5500 2800
 	1    0    0    -1
 $EndComp
@@
 F 0 "TP12" H 7700 2900 50  0000 C CNN
 F 1 "RAIL_OR_SAFETY_TEST_POINT" H 7700 2700 50  0000 C CNN
+F 2 "" H 7600 2800 50  0001 C CNN
+F 3 "" H 7600 2800 50  0001 C CNN
+	1    7600 2800
 	1    0    0    -1
 $EndComp
@@
 F 0 "TP13" H 1400 3700 50  0000 C CNN
 F 1 "RAIL_OR_SAFETY_TEST_POINT" H 1400 3500 50  0000 C CNN
+F 2 "" H 1300 3600 50  0001 C CNN
+F 3 "" H 1300 3600 50  0001 C CNN
+	1    1300 3600
 	1    0    0    -1
 $EndComp
@@
 F 0 "TP14" H 3500 3700 50  0000 C CNN
 F 1 "RAIL_OR_SAFETY_TEST_POINT" H 3500 3500 50  0000 C CNN
+F 2 "" H 3400 3600 50  0001 C CNN
+F 3 "" H 3400 3600 50  0001 C CNN
+	1    3400 3600
 	1    0    0    -1
 $EndComp
@@
 F 0 "TP15" H 5600 3700 50  0000 C CNN
 F 1 "RAIL_OR_SAFETY_TEST_POINT" H 5600 3500 50  0000 C CNN
+F 2 "" H 5500 3600 50  0001 C CNN
+F 3 "" H 5500 3600 50  0001 C CNN
+	1    5500 3600
 	1    0    0    -1
 $EndComp
@@
 F 0 "TP16" H 7700 3700 50  0000 C CNN
 F 1 "RAIL_OR_SAFETY_TEST_POINT" H 7700 3500 50  0000 C CNN
-	1    0    0    -1
-$EndComp
-Text Label 700 5600 0    50   ~ 0
-TP_ALL_RAILS
-Text Label 700 5840 0    50   ~ 0
-TP_USB_PRESENT
-Text Label 700 6080 0    50   ~ 0
-TP_BATTERY_VALID
-Text Label 700 6320 0    50   ~ 0
-TP_SAFETY_POWER_GOOD
-Text Label 700 6560 0    50   ~ 0
-TP_EDA_ANALOG_GOOD
-Text Label 700 6800 0    50   ~ 0
-TP_SYNC_BOTH_SIDES
-Text Label 700 7040 0    50   ~ 0
-TP_SD_ACTIVITY
-Text Label 700 7280 0    50   ~ 0
-FAULT_INJECTION
+F 2 "" H 7600 3600 50  0001 C CNN
+F 3 "" H 7600 3600 50  0001 C CNN
+	1    7600 3600
+	1    0    0    -1
+$EndComp
 Text Notes 600 400 0    50   ~ 0
 ENGINEERING REVIEW ONLY - NOT FOR HUMAN CONNECTION
+Text Notes 700 5600 0    50   ~ 0
+NET:TP_ALL_RAILS
+Text Notes 700 5850 0    50   ~ 0
+NET:TP_USB_PRESENT
+Text Notes 700 6100 0    50   ~ 0
+NET:TP_BATTERY_VALID
+Text Notes 700 6350 0    50   ~ 0
+NET:TP_SAFETY_POWER_GOOD
+Text Notes 700 6600 0    50   ~ 0
+NET:TP_EDA_ANALOG_GOOD
+Text Notes 700 6850 0    50   ~ 0
+NET:TP_SYNC_BOTH_SIDES
+Text Notes 700 7100 0    50   ~ 0
+NET:TP_SD_ACTIVITY
+Text Notes 700 7350 0    50   ~ 0
+NET:FAULT_INJECTION
 Text Notes 6000 5600 0    50   ~ 0
 NO LAB GROUND ON BAT_HUMAN TEST POINT
