File: hardware/circle-ppg/legacy/00_ppg_root.sch (KiCad schematic (older format))
At the start: 10 parts, among them U101 MAX30102, U102 1V8_LOW_NOISE_LDO, U103 I2C_LEVEL_TRANSLATOR, U104 AT24CS02, U105 LIS2DW12

Commit message: Make every CIRCLE review claim reproducible
Validate and export the architecture-level schematics with KiCad 10.0.5, add zero-violation ERC gates, engineering documentation, and one-command evidence hashing.

Constraint: KiCad CLI does not import legacy .sch into native .kicad_sch

Rejected: Hand-written native S-expressions | would create unvalidated CAD

Confidence: medium

Scope-risk: broad

Reversibility: clean

Directive: Treat NET annotations as architecture interfaces, not fabrication-ready connectivity

Tested: py -3.11 tools/verify_release.py; 30 tests; KiCad 10.0.5 ERC/BOM/PDF/SVG/netlist exports

Not-tested: Native conversion, PCB layout, footprints, powered electrodes, human connection, EMC, or regulatory compliance
Other:
- note added: "NET:PPG_3V3"
- note added: "NET:PPG_INT"
- note added: "NET:PPG_LED_GND"
- note added: "NET:PPG_LED_PWR"
- note added: "NET:PPG_LOGIC_GND"
- note added: "NET:PPG_SCL_3V3"
- note added: "NET:PPG_SDA_3V3"
Changed lines of the file:
@@
 Sheet 1 1
 Title "PPG contact board"
+Date "2026-08-14"
+Rev "A"
+Comp "Vers3Dynamics"
 Comment1 "ENGINEERING REVIEW ONLY - NOT FOR HUMAN CONNECTION"
+Comment2 "Generated artifact - edit manifest/generator"
+Comment3 ""
+Comment4 ""
 $EndDescr
 $Comp
@@
 F 0 "U101" H 1400 1300 50  0000 C CNN
 F 1 "MAX30102" H 1400 1100 50  0000 C CNN
+F 2 "" H 1300 1200 50  0001 C CNN
+F 3 "" H 1300 1200 50  0001 C CNN
+	1    1300 1200
 	1    0    0    -1
 $EndComp
@@
 F 0 "U102" H 3500 1300 50  0000 C CNN
 F 1 "1V8_LOW_NOISE_LDO" H 3500 1100 50  0000 C CNN
+F 2 "" H 3400 1200 50  0001 C CNN
+F 3 "" H 3400 1200 50  0001 C CNN
+	1    3400 1200
 	1    0    0    -1
 $EndComp
@@
 F 0 "U103" H 5600 1300 50  0000 C CNN
 F 1 "I2C_LEVEL_TRANSLATOR" H 5600 1100 50  0000 C CNN
+F 2 "" H 5500 1200 50  0001 C CNN
+F 3 "" H 5500 1200 50  0001 C CNN
+	1    5500 1200
 	1    0    0    -1
 $EndComp
@@
 F 0 "U104" H 7700 1300 50  0000 C CNN
 F 1 "AT24CS02" H 7700 1100 50  0000 C CNN
+F 2 "" H 7600 1200 50  0001 C CNN
+F 3 "" H 7600 1200 50  0001 C CNN
+	1    7600 1200
 	1    0    0    -1
 $EndComp
@@
 F 0 "U105" H 1400 2100 50  0000 C CNN
 F 1 "LIS2DW12" H 1400 1900 50  0000 C CNN
+F 2 "" H 1300 2000 50  0001 C CNN
+F 3 "" H 1300 2000 50  0001 C CNN
+	1    1300 2000
 	1    0    0    -1
 $EndComp
@@
 F 0 "D101" H 3500 2100 50  0000 C CNN
 F 1 "PPG_CABLE_ESD" H 3500 1900 50  0000 C CNN
+F 2 "" H 3400 2000 50  0001 C CNN
+F 3 "" H 3400 2000 50  0001 C CNN
+	1    3400 2000
 	1    0    0    -1
 $EndComp
@@
 F 0 "R101" H 5600 2100 50  0000 C CNN
 F 1 "I2C_DAMPING" H 5600 1900 50  0000 C CNN
+F 2 "" H 5500 2000 50  0001 C CNN
+F 3 "" H 5500 2000 50  0001 C CNN
+	1    5500 2000
 	1    0    0    -1
 $EndComp
@@
 F 0 "R102" H 7700 2100 50  0000 C CNN
 F 1 "I2C_DAMPING" H 7700 1900 50  0000 C CNN
+F 2 "" H 7600 2000 50  0001 C CNN
+F 3 "" H 7600 2000 50  0001 C CNN
+	1    7600 2000
 	1    0    0    -1
 $EndComp
@@
 F 0 "C101" H 1400 2900 50  0000 C CNN
 F 1 "LOGIC_DECOUPLING" H 1400 2700 50  0000 C CNN
+F 2 "" H 1300 2800 50  0001 C CNN
+F 3 "" H 1300 2800 50  0001 C CNN
+	1    1300 2800
 	1    0    0    -1
 $EndComp
@@
 F 0 "C102" H 3500 2900 50  0000 C CNN
 F 1 "LED_FILTER" H 3500 2700 50  0000 C CNN
+F 2 "" H 3400 2800 50  0001 C CNN
+F 3 "" H 3400 2800 50  0001 C CNN
+	1    3400 2800
 	1    0    0    -1
 $EndComp
-Text Label 700 5840 0    50   ~ 0
-PPG_3V3
-Text Label 700 6080 0    50   ~ 0
-PPG_LED_PWR
-Text Label 700 6320 0    50   ~ 0
-PPG_LOGIC_GND
-Text Label 700 6560 0    50   ~ 0
-PPG_LED_GND
-Text Label 700 6800 0    50   ~ 0
-PPG_SDA_3V3
-Text Label 700 7040 0    50   ~ 0
-PPG_SCL_3V3
-Text Label 700 7280 0    50   ~ 0
-PPG_INT
 Text Notes 600 400 0    50   ~ 0
 ENGINEERING REVIEW ONLY - NOT FOR HUMAN CONNECTION
 Text Notes 700 5600 0    50   ~ 0
 MAX30102 RAW RED/IR ONLY
+Text Notes 700 5850 0    50   ~ 0
+NET:PPG_3V3
+Text Notes 700 6100 0    50   ~ 0
+NET:PPG_LED_PWR
+Text Notes 700 6350 0    50   ~ 0
+NET:PPG_LOGIC_GND
+Text Notes 700 6600 0    50   ~ 0
+NET:PPG_LED_GND
+Text Notes 700 6850 0    50   ~ 0
+NET:PPG_SDA_3V3
+Text Notes 700 7100 0    50   ~ 0
+NET:PPG_SCL_3V3
+Text Notes 700 7350 0    50   ~ 0
+NET:PPG_INT
 Text Notes 6000 5600 0    50   ~ 0
 AT24CS02 BOARD ID
-Text Notes 6000 5840 0    50   ~ 0
+Text Notes 6000 5850 0    50   ~ 0
 LIS2DW12 DNI
-Text Notes 6000 6080 0    50   ~ 0
+Text Notes 6000 6100 0    50   ~ 0
 OPTICAL KEEP-OUT AND AMBIENT-LIGHT EXCLUSION
 $EndSCHEMATC
